File: Hardware/PCB_Proiect_v290.brd (EAGLE design)
At the start: 170.2 x 111.5 mm, 103 parts, among them IC1 XC6220A331MR-G, IC2 BD5229G-TR, J1 112A-TAAR-R03_ATTEND, J2 QWIIC_RIGHT_ANGLE, J3 FH34SRJ-24S-0.5SH_99_, J4 SAMACSYS_PARTS_USB4110-GF-A, Q1 20V/4.2A/52mΩ/1.4W, Q2 SI1308EDL-T1-GE3, U1 ESP32-C6-WROOM-1-N8, U2 MAX17048G+T10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

Commit message: For #3
Parts:
- moved R_CHANGE 0.20 mm to (44.7, 108.3)
- moved R_RESET 0.10 mm to (60.3, 108.1)
